File: Hardware/Boards/Input_Signal_Conditioner/Input_Signal_Conditioner.sch (KiCad schematic (older format))
At the start: 19 parts, among them U1 LTC6256CMS8#PBF

Commit message: Assigned PCB footprints to ISC. Started layout of the PCB, traces still need to be routed.
Parts:
- removed J?: Conn_01x02, symbol Connector_Generic:Conn_01x02
- added J1, J2: Conn_01x01, Connector_PinSocket_2.54mm:PinSocket_1x01_P2.54mm_Vertical, symbol Connector_Generic:Conn_01x01
- C1, C2, C3, C4, C5: footprint (none) -> Capacitor_SMD:C_1206_3216Metric
- C6: renamed from C?; footprint (none) -> Capacitor_SMD:C_1206_3216Metric
- J3: renamed from J?; footprint (none) -> Connector_PinSocket_2.54mm:PinSocket_1x05_P2.54mm_Vertical
- J4: renamed from J?; footprint (none) -> Connector_PinSocket_2.54mm:PinSocket_1x03_P2.54mm_Vertical
- R1, R2, R3, R4, R5, R6, R7, R8, R9: footprint (none) -> Resistor_SMD:R_1206_3216Metric
- U1: footprint (none) -> LTC6256CMS8PBF:LTC6256CMS8-PBF
Connections:
- net 3.3V: now also J3.5 (Pin_5); no longer J3.1 (Pin_1)
- net ADC_IN: now also J3.2 (Pin_2); no longer J3.4 (Pin_4)
- net GND: now also J3.1 (Pin_1), J3.4 (Pin_4), J2.1 (Pin_1); no longer J3.2 (Pin_2), J3.5 (Pin_5)
- net MIC_IN+: now also J1.1 (Pin_1)
- net AMP_IN: now reaches J4.3 (Pin_3), R3.1, U1.3 (+)
- net FILT_IN: now reaches R5.1, R6.2, U1.1
- net FILT_OUT: now reaches C5.1, R8.2, U1.6 (-), U1.7
Changed lines of the file:
@@
 F 0 "C2" H 3640 4171 50  0000 L CNN
 F 1 "4.7u" H 3640 4080 50  0000 L CNN
-F 2 "" H 3563 3975 50  0001 C CNN
+F 2 "Capacitor_SMD:C_1206_3216Metric" H 3563 3975 50  0001 C CNN
 F 3 "~" H 3525 4125 50  0001 C CNN
 	1    3525 4125
@@
 F 0 "C1" V 2023 2775 50  0000 C CNN
 F 1 "220n" V 2114 2775 50  0000 C CNN
-F 2 "" H 2313 2625 50  0001 C CNN
+F 2 "Capacitor_SMD:C_1206_3216Metric" H 2313 2625 50  0001 C CNN
 F 3 "~" H 2275 2775 50  0001 C CNN
 	1    2275 2775
@@
 F 0 "C3" H 4565 4521 50  0000 L CNN
 F 1 "4.7u" H 4565 4430 50  0000 L CNN
-F 2 "" H 4488 4325 50  0001 C CNN
+F 2 "Capacitor_SMD:C_1206_3216Metric" H 4488 4325 50  0001 C CNN
 F 3 "~" H 4450 4475 50  0001 C CNN
 	1    4450 4475
@@
 F 0 "R4" H 4518 3996 50  0000 L CNN
 F 1 "1K" H 4518 3905 50  0000 L CNN
-F 2 "" V 4490 3940 50  0001 C CNN
+F 2 "Resistor_SMD:R_1206_3216Metric" V 4490 3940 50  0001 C CNN
 F 3 "~" H 4450 3950 50  0001 C CNN
 	1    4450 3950
@@
 F 0 "R5" V 5100 3725 50  0000 C CNN
 F 1 "50K" V 5175 3750 50  0000 C CNN
-F 2 "" V 5040 3615 50  0001 C CNN
+F 2 "Resistor_SMD:R_1206_3216Metric" V 5040 3615 50  0001 C CNN
 F 3 "~" H 5000 3625 50  0001 C CNN
 	1    5000 3625
@@
 F 0 "R7" H 6268 3496 50  0000 L CNN
 F 1 "11.25K" H 6268 3405 50  0000 L CNN
-F 2 "" V 6240 3440 50  0001 C CNN
+F 2 "Resistor_SMD:R_1206_3216Metric" V 6240 3440 50  0001 C CNN
 F 3 "~" H 6200 3450 50  0001 C CNN
 	1    6200 3450
@@
 F 0 "C4" H 6315 4196 50  0000 L CNN
 F 1 "2.5n" H 6315 4105 50  0000 L CNN
-F 2 "" H 6238 4000 50  0001 C CNN
+F 2 "Capacitor_SMD:C_1206_3216Metric" H 6238 4000 50  0001 C CNN
 F 3 "~" H 6200 4150 50  0001 C CNN
 	1    6200 4150
@@
 F 0 "R6" V 5645 3100 50  0000 C CNN
 F 1 "11.25K" V 5736 3100 50  0000 C CNN
-F 2 "" V 5890 3090 50  0001 C CNN
+F 2 "Resistor_SMD:R_1206_3216Metric" V 5890 3090 50  0001 C CNN
 F 3 "~" H 5850 3100 50  0001 C CNN
 	1    5850 3100
@@
 F 0 "C5" V 6725 3175 50  0000 L CNN
 F 1 "5n" V 6800 3175 50  0000 L CNN
-F 2 "" H 6963 2950 50  0001 C CNN
+F 2 "Capacitor_SMD:C_1206_3216Metric" H 6963 2950 50  0001 C CNN
 F 3 "~" H 6925 3100 50  0001 C CNN
 	1    6925 3100
@@
 F 0 "U1" H 4883 3100 50  0001 L CNN
 F 1 "LTC6256CMS8#PBF" H 4883 3055 50  0001 L CNN
-F 2 "" H 4925 3100 50  0001 C CNN
+F 2 "LTC6256CMS8PBF:LTC6256CMS8-PBF" H 4925 3100 50  0001 C CNN
 F 3 "https://www.analog.com/media/en/technical-documentation/data-sheets/ADA4807-1_4807-2_4807-4.pdf" H 4925 3100 50  0001 C CNN
 	3    4925 3100
@@
 F 0 "U1" H 7025 4217 50  0000 C CNN
 F 1 "LTC6256CMS8#PBF" H 7025 4126 50  0000 C CNN
-F 2 "" H 7025 3850 50  0001 C CNN
+F 2 "LTC6256CMS8PBF:LTC6256CMS8-PBF" H 7025 3850 50  0001 C CNN
 F 3 "https://www.analog.com/media/en/technical-documentation/data-sheets/ADA4807-1_4807-2_4807-4.pdf" H 7025 3850 50  0001 C CNN
 	2    7025 3850
@@
 F 0 "U1" H 4300 3450 50  0000 C CNN
 F 1 "LTC6256CMS8#PBF" H 4425 3375 50  0000 C CNN
-F 2 "" H 4925 3100 50  0001 C CNN
+F 2 "LTC6256CMS8PBF:LTC6256CMS8-PBF" H 4925 3100 50  0001 C CNN
 F 3 "https://www.analog.com/media/en/technical-documentation/data-sheets/ADA4807-1_4807-2_4807-4.pdf" H 4925 3100 50  0001 C CNN
 	1    4925 3100
@@
 F 0 "R1" H 2993 3596 50  0000 L CNN
 F 1 "50K" H 2993 3505 50  0000 L CNN
-F 2 "" V 2965 3540 50  0001 C CNN
+F 2 "Resistor_SMD:R_1206_3216Metric" V 2965 3540 50  0001 C CNN
 F 3 "~" H 2925 3550 50  0001 C CNN
 	1    2925 3550
@@
 F 0 "R2" H 2993 4171 50  0000 L CNN
 F 1 "50K" H 2993 4080 50  0000 L CNN
-F 2 "" V 2965 4115 50  0001 C CNN
+F 2 "Resistor_SMD:R_1206_3216Metric" V 2965 4115 50  0001 C CNN
 F 3 "~" H 2925 4125 50  0001 C CNN
 	1    2925 4125
@@
 F 0 "R3" H 3593 3421 50  0000 L CNN
 F 1 "100K" H 3593 3330 50  0000 L CNN
-F 2 "" V 3565 3365 50  0001 C CNN
+F 2 "Resistor_SMD:R_1206_3216Metric" V 3565 3365 50  0001 C CNN
 F 3 "~" H 3525 3375 50  0001 C CNN
 	1    3525 3375
@@
 F 0 "R8" V 7870 3100 50  0000 C CNN
 F 1 "0" V 7961 3100 50  0000 C CNN
-F 2 "" V 8115 3090 50  0001 C CNN
+F 2 "Resistor_SMD:R_1206_3216Metric" V 8115 3090 50  0001 C CNN
 F 3 "~" H 8075 3100 50  0001 C CNN
 	1    8075 3100
@@
 F 0 "R9" H 8600 3325 50  0000 C CNN
 F 1 "INF" H 8550 3400 50  0000 C CNN
-F 2 "" V 8415 3340 50  0001 C CNN
+F 2 "Resistor_SMD:R_1206_3216Metric" V 8415 3340 50  0001 C CNN
 F 3 "~" H 8375 3350 50  0001 C CNN
 	1    8375 3350
@@
 BYPASS SWITCH SPDT PINS\n
 $Comp
-L Connector_Generic:Conn_01x03 J?
+L Connector_Generic:Conn_01x03 J4
 U 1 1 5F90B259
 P 3225 2775
-F 0 "J?" H 3305 2817 50  0000 L CNN
+F 0 "J4" H 3305 2817 50  0000 L CNN
 F 1 "Conn_01x03" H 3305 2726 50  0000 L CNN
-F 2 "" H 3225 2775 50  0001 C CNN
+F 2 "Connector_PinSocket_2.54mm:PinSocket_1x03_P2.54mm_Vertical" H 3225 2775 50  0001 C CNN
 F 3 "~" H 3225 2775 50  0001 C CNN
 	1    3225 2775
@@
 Connection ~ 3525 3000
 $Comp
-L Connector_Generic:Conn_01x02 J?
-U 1 1 5F91649E
-P 2375 5775
-F 0 "J?" H 2455 5767 50  0000 L CNN
-F 1 "Conn_01x02" H 2455 5676 50  0000 L CNN
-F 2 "" H 2375 5775 50  0001 C CNN
-F 3 "~" H 2375 5775 50  0001 C CNN
-	1    2375 5775
-	1    0    0    -1
-$EndComp
-$Comp
-L Connector_Generic:Conn_01x05 J?
+L Connector_Generic:Conn_01x05 J3
 U 1 1 5F91BE34
 P 3900 5925
-F 0 "J?" H 3980 5967 50  0000 L CNN
+F 0 "J3" H 3980 5967 50  0000 L CNN
 F 1 "Conn_01x05" H 3980 5876 50  0000 L CNN
-F 2 "" H 3900 5925 50  0001 C CNN
+F 2 "Connector_PinSocket_2.54mm:PinSocket_1x05_P2.54mm_Vertical" H 3900 5925 50  0001 C CNN
 F 3 "~" H 3900 5925 50  0001 C CNN
 	1    3900 5925
-	-1   0    0    1
+	-1   0    0    -1
 $EndComp
 Wire Wire Line
 	2175 5775 1800 5775
 Wire Wire Line
-	2175 5875 2075 5875
-Wire Wire Line
-	2075 5875 2075 5975
-Wire Wire Line
-	2075 5975 1800 5975
+	2175 6100 2075 6100
+Wire Wire Line
+	2075 6100 2075 6200
+Wire Wire Line
+	2075 6100 1800 6100
 Text GLabel 1800 5775 0    50   Input ~ 0
 MIC_IN+
-Text GLabel 1800 5975 0    50   Input ~ 0
+Text GLabel 1800 6100 0    50   Input ~ 0
 MIC_IN-
 $Comp
-L power:GND #PWR?
+L power:GND #PWR07
 U 1 1 5F922B0D
-P 2075 6075
-F 0 "#PWR?" H 2075 5825 50  0001 C CNN
-F 1 "GND" H 2080 5902 50  0000 C CNN
-F 2 "" H 2075 6075 50  0001 C CNN
-F 3 "" H 2075 6075 50  0001 C CNN
-	1    2075 6075
-	1    0    0    -1
-$EndComp
-Wire Wire Line
-	2075 6075 2075 5975
-Connection ~ 2075 5975
+P 2075 6200
+F 0 "#PWR07" H 2075 5950 50  0001 C CNN
+F 1 "GND" H 2080 6027 50  0000 C CNN
+F 2 "" H 2075 6200 50  0001 C CNN
+F 3 "" H 2075 6200 50  0001 C CNN
+	1    2075 6200
+	1    0    0    -1
+$EndComp
 Text GLabel 4775 6225 2    50   Input ~ 0
 3.3V
@@
 	4250 6225 4600 6225
 $Comp
-L power:GND #PWR?
+L power:GND #PWR08
 U 1 1 5F95E124
 P 4175 6400
-F 0 "#PWR?" H 4175 6150 50  0001 C CNN
+F 0 "#PWR08" H 4175 6150 50  0001 C CNN
 F 1 "GND" H 4180 6227 50  0000 C CNN
 F 2 "" H 4175 6400 50  0001 C CNN
@@
 	4600 6225 4775 6225
 $Comp
-L Device:C C?
+L Device:C C6
 U 1 1 5F9621B2
 P 4600 6700
-F 0 "C?" H 4715 6746 50  0000 L CNN
+F 0 "C6" H 4715 6746 50  0000 L CNN
 F 1 "0.1u" H 4715 6655 50  0000 L CNN
-F 2 "" H 4638 6550 50  0001 C CNN
+F 2 "Capacitor_SMD:C_1206_3216Metric" H 4638 6550 50  0001 C CNN
 F 3 "~" H 4600 6700 50  0001 C CNN
 	1    4600 6700
@@
 $EndComp
 $Comp
-L power:GND #PWR?
+L power:GND #PWR09
 U 1 1 5F963219
 P 4600 6950
-F 0 "#PWR?" H 4600 6700 50  0001 C CNN
+F 0 "#PWR09" H 4600 6700 50  0001 C CNN
 F 1 "GND" H 4605 6777 50  0000 C CNN
 F 2 "" H 4600 6950 50  0001 C CNN
@@
 Wire Wire Line
 	4600 6950 4600 6850
+$Comp
+L power:PWR_FLAG #FLG0101
+U 1 1 5F936862
+P 9400 5825
+F 0 "#FLG0101" H 9400 5900 50  0001 C CNN
+F 1 "PWR_FLAG" H 9400 5998 50  0000 C CNN
+F 2 "" H 9400 5825 50  0001 C CNN
+F 3 "~" H 9400 5825 50  0001 C CNN
+	1    9400 5825
+	1    0    0    -1
+$EndComp
+$Comp
+L power:GND #PWR0101
+U 1 1 5F936CB6
+P 9400 6000
+F 0 "#PWR0101" H 9400 5750 50  0001 C CNN
+F 1 "GND" H 9405 5827 50  0000 C CNN
+F 2 "" H 9400 6000 50  0001 C CNN
+F 3 "" H 9400 6000 50  0001 C CNN
+	1    9400 6000
+	1    0    0    -1
+$EndComp
+$Comp
+L power:PWR_FLAG #FLG0102
+U 1 1 5F93ABBE
+P 8800 6025
+F 0 "#FLG0102" H 8800 6100 50  0001 C CNN
+F 1 "PWR_FLAG" H 8800 6198 50  0000 C CNN
+F 2 "" H 8800 6025 50  0001 C CNN
+F 3 "~" H 8800 6025 50  0001 C CNN
+	1    8800 6025
+	-1   0    0    1
+$EndComp
+Text GLabel 8800 5825 1    50   Input ~ 0
+3.3V
+Wire Wire Line
+	8800 6025 8800 5825
+Wire Wire Line
+	9400 6000 9400 5825
+$Comp
+L Connector_Generic:Conn_01x01 J1
+U 1 1 5F94CBF1
+P 2375 5775
+F 0 "J1" H 2455 5817 50  0000 L CNN
+F 1 "Conn_01x01" H 2455 5726 50  0000 L CNN
+F 2 "Connector_PinSocket_2.54mm:PinSocket_1x01_P2.54mm_Vertical" H 2375 5775 50  0001 C CNN
+F 3 "~" H 2375 5775 50  0001 C CNN
+	1    2375 5775
+	1    0    0    -1
+$EndComp
+$Comp
+L Connector_Generic:Conn_01x01 J2
+U 1 1 5F9504CB
+P 2375 6100
+F 0 "J2" H 2455 6142 50  0000 L CNN
+F 1 "Conn_01x01" H 2455 6051 50  0000 L CNN
+F 2 "Connector_PinSocket_2.54mm:PinSocket_1x01_P2.54mm_Vertical" H 2375 6100 50  0001 C CNN
+F 3 "~" H 2375 6100 50  0001 C CNN
+	1    2375 6100
+	1    0    0    -1
+$EndComp
+Connection ~ 2075 6100
+Text Label 7500 3100 0    50   ~ 0
+FILT_OUT
+Text Label 5350 3100 0    50   ~ 0
+FILT_IN
+Text Label 3850 3000 0    50   ~ 0
+AMP_IN
 $EndSCHEMATC

Commit message: Redesigned the ISC LPF filter to a new cutoff frequency. Also began documentation of the ISC design. Updated the LTSpice simulation of the ISC to reflect LPF changes. Choose an Op-amp for the design.
Connections:
- net ADC_IN: now also J3.3 (Pin_3); no longer J3.2 (Pin_2)
- net BYPASS: now also J3.2 (Pin_2); no longer J3.3 (Pin_3)
Changed lines of the file:
@@
 Text GLabel 4775 6100 2    50   Input ~ 0
 GND
+Text GLabel 4775 5825 2    50   Output ~ 0
+BYPASS
 Text GLabel 4775 5950 2    50   Output ~ 0
-BYPASS
-Text GLabel 4775 5825 2    50   Output ~ 0
 ADC_IN
 Text GLabel 4775 5700 2    50   Input ~ 0

Commit message: Redid the layout of the PCB to be THT components. Layout needs review, then it is ready to print.
Parts:
- C1, C3, C6: footprint Capacitor_SMD:C_1206_3216Metric -> Capacitor_THT:C_Disc_D7.5mm_W4.4mm_P5.00mm
- C2: value 4.7u -> 4.7n; footprint Capacitor_SMD:C_1206_3216Metric -> Capacitor_THT:C_Disc_D7.5mm_W4.4mm_P5.00mm
- C4: value 2.5n -> 680p; footprint Capacitor_SMD:C_1206_3216Metric -> Capacitor_THT:C_Disc_D7.5mm_W4.4mm_P5.00mm
- C5: value 5n -> 1.5n; footprint Capacitor_SMD:C_1206_3216Metric -> Capacitor_THT:C_Disc_D7.5mm_W4.4mm_P5.00mm
- R1, R2, R3, R4, R6, R8, R9: footprint Resistor_SMD:R_1206_3216Metric -> Resistor_THT:R_Axial_DIN0207_L6.3mm_D2.5mm_P10.16mm_Horizontal
- R5: value 50K -> 11K; footprint Resistor_SMD:R_1206_3216Metric -> Resistor_THT:R_Axial_DIN0207_L6.3mm_D2.5mm_P10.16mm_Horizontal
- R7: value 11.25K -> 14.3K; footprint Resistor_SMD:R_1206_3216Metric -> Resistor_THT:R_Axial_DIN0207_L6.3mm_D2.5mm_P10.16mm_Horizontal
- U1: value LTC6256CMS8#PBF -> MCP6272; footprint LTC6256CMS8PBF:LTC6256CMS8-PBF -> Package_DIP:DIP-8_W7.62mm
Changed lines of the file:
@@
 P 3525 4125
 F 0 "C2" H 3640 4171 50  0000 L CNN
-F 1 "4.7u" H 3640 4080 50  0000 L CNN
-F 2 "Capacitor_SMD:C_1206_3216Metric" H 3563 3975 50  0001 C CNN
+F 1 "4.7n" H 3640 4080 50  0000 L CNN
+F 2 "Capacitor_THT:C_Disc_D7.5mm_W4.4mm_P5.00mm" H 3563 3975 50  0001 C CNN
 F 3 "~" H 3525 4125 50  0001 C CNN
 	1    3525 4125
@@
 F 0 "C1" V 2023 2775 50  0000 C CNN
 F 1 "220n" V 2114 2775 50  0000 C CNN
-F 2 "Capacitor_SMD:C_1206_3216Metric" H 2313 2625 50  0001 C CNN
+F 2 "Capacitor_THT:C_Disc_D7.5mm_W4.4mm_P5.00mm" H 2313 2625 50  0001 C CNN
 F 3 "~" H 2275 2775 50  0001 C CNN
 	1    2275 2775
@@
 F 0 "C3" H 4565 4521 50  0000 L CNN
 F 1 "4.7u" H 4565 4430 50  0000 L CNN
-F 2 "Capacitor_SMD:C_1206_3216Metric" H 4488 4325 50  0001 C CNN
+F 2 "Capacitor_THT:C_Disc_D7.5mm_W4.4mm_P5.00mm" H 4488 4325 50  0001 C CNN
 F 3 "~" H 4450 4475 50  0001 C CNN
 	1    4450 4475
@@
 F 0 "R4" H 4518 3996 50  0000 L CNN
 F 1 "1K" H 4518 3905 50  0000 L CNN
-F 2 "Resistor_SMD:R_1206_3216Metric" V 4490 3940 50  0001 C CNN
+F 2 "Resistor_THT:R_Axial_DIN0207_L6.3mm_D2.5mm_P10.16mm_Horizontal" V 4490 3940 50  0001 C CNN
 F 3 "~" H 4450 3950 50  0001 C CNN
 	1    4450 3950
@@
 P 5000 3625
 F 0 "R5" V 5100 3725 50  0000 C CNN
-F 1 "50K" V 5175 3750 50  0000 C CNN
-F 2 "Resistor_SMD:R_1206_3216Metric" V 5040 3615 50  0001 C CNN
+F 1 "11K" V 5175 3750 50  0000 C CNN
+F 2 "Resistor_THT:R_Axial_DIN0207_L6.3mm_D2.5mm_P10.16mm_Horizontal" V 5040 3615 50  0001 C CNN
 F 3 "~" H 5000 3625 50  0001 C CNN
 	1    5000 3625
@@
 P 6200 3450
 F 0 "R7" H 6268 3496 50  0000 L CNN
-F 1 "11.25K" H 6268 3405 50  0000 L CNN
-F 2 "Resistor_SMD:R_1206_3216Metric" V 6240 3440 50  0001 C CNN
+F 1 "14.3K" H 6268 3405 50  0000 L CNN
+F 2 "Resistor_THT:R_Axial_DIN0207_L6.3mm_D2.5mm_P10.16mm_Horizontal" V 6240 3440 50  0001 C CNN
 F 3 "~" H 6200 3450 50  0001 C CNN
 	1    6200 3450
@@
 P 6200 4150
 F 0 "C4" H 6315 4196 50  0000 L CNN
-F 1 "2.5n" H 6315 4105 50  0000 L CNN
-F 2 "Capacitor_SMD:C_1206_3216Metric" H 6238 4000 50  0001 C CNN
+F 1 "680p" H 6315 4105 50  0000 L CNN
+F 2 "Capacitor_THT:C_Disc_D7.5mm_W4.4mm_P5.00mm" H 6238 4000 50  0001 C CNN
 F 3 "~" H 6200 4150 50  0001 C CNN
 	1    6200 4150
@@
 F 0 "R6" V 5645 3100 50  0000 C CNN
 F 1 "11.25K" V 5736 3100 50  0000 C CNN
-F 2 "Resistor_SMD:R_1206_3216Metric" V 5890 3090 50  0001 C CNN
+F 2 "Resistor_THT:R_Axial_DIN0207_L6.3mm_D2.5mm_P10.16mm_Horizontal" V 5890 3090 50  0001 C CNN
 F 3 "~" H 5850 3100 50  0001 C CNN
 	1    5850 3100
@@
 P 6925 3100
 F 0 "C5" V 6725 3175 50  0000 L CNN
-F 1 "5n" V 6800 3175 50  0000 L CNN
-F 2 "Capacitor_SMD:C_1206_3216Metric" H 6963 2950 50  0001 C CNN
+F 1 "1.5n" V 6800 3175 50  0000 L CNN
+F 2 "Capacitor_THT:C_Disc_D7.5mm_W4.4mm_P5.00mm" H 6963 2950 50  0001 C CNN
 F 3 "~" H 6925 3100 50  0001 C CNN
 	1    6925 3100
@@
 P 4925 3100
 F 0 "U1" H 4883 3100 50  0001 L CNN
-F 1 "LTC6256CMS8#PBF" H 4883 3055 50  0001 L CNN
-F 2 "LTC6256CMS8PBF:LTC6256CMS8-PBF" H 4925 3100 50  0001 C CNN
-F 3 "https://www.analog.com/media/en/technical-documentation/data-sheets/ADA4807-1_4807-2_4807-4.pdf" H 4925 3100 50  0001 C CNN
+F 1 "MCP6272" H 4883 3055 50  0001 L CNN
+F 2 "Package_DIP:DIP-8_W7.62mm" H 4925 3100 50  0001 C CNN
+F 3 "https://ww1.microchip.com/downloads/en/DeviceDoc/20001810G.pdf" H 4925 3100 50  0001 C CNN
 	3    4925 3100
 	1    0    0    -1
@@
 P 7025 3850
 F 0 "U1" H 7025 4217 50  0000 C CNN
-F 1 "LTC6256CMS8#PBF" H 7025 4126 50  0000 C CNN
-F 2 "LTC6256CMS8PBF:LTC6256CMS8-PBF" H 7025 3850 50  0001 C CNN
-F 3 "https://www.analog.com/media/en/technical-documentation/data-sheets/ADA4807-1_4807-2_4807-4.pdf" H 7025 3850 50  0001 C CNN
+F 1 "MCP6272" H 7025 4126 50  0000 C CNN
+F 2 "Package_DIP:DIP-8_W7.62mm" H 7025 3850 50  0001 C CNN
+F 3 "https://ww1.microchip.com/downloads/en/DeviceDoc/20001810G.pdf" H 7025 3850 50  0001 C CNN
 	2    7025 3850
 	1    0    0    -1
@@
 P 4925 3100
 F 0 "U1" H 4300 3450 50  0000 C CNN
-F 1 "LTC6256CMS8#PBF" H 4425 3375 50  0000 C CNN
-F 2 "LTC6256CMS8PBF:LTC6256CMS8-PBF" H 4925 3100 50  0001 C CNN
-F 3 "https://www.analog.com/media/en/technical-documentation/data-sheets/ADA4807-1_4807-2_4807-4.pdf" H 4925 3100 50  0001 C CNN
+F 1 "MCP6272" H 4425 3375 50  0000 C CNN
+F 2 "Package_DIP:DIP-8_W7.62mm" H 4925 3100 50  0001 C CNN
+F 3 "https://ww1.microchip.com/downloads/en/DeviceDoc/20001810G.pdf" H 4925 3100 50  0001 C CNN
 	1    4925 3100
 	1    0    0    -1
@@
 F 0 "R1" H 2993 3596 50  0000 L CNN
 F 1 "50K" H 2993 3505 50  0000 L CNN
-F 2 "Resistor_SMD:R_1206_3216Metric" V 2965 3540 50  0001 C CNN
+F 2 "Resistor_THT:R_Axial_DIN0207_L6.3mm_D2.5mm_P10.16mm_Horizontal" V 2965 3540 50  0001 C CNN
 F 3 "~" H 2925 3550 50  0001 C CNN
 	1    2925 3550
@@
 F 0 "R2" H 2993 4171 50  0000 L CNN
 F 1 "50K" H 2993 4080 50  0000 L CNN
-F 2 "Resistor_SMD:R_1206_3216Metric" V 2965 4115 50  0001 C CNN
+F 2 "Resistor_THT:R_Axial_DIN0207_L6.3mm_D2.5mm_P10.16mm_Horizontal" V 2965 4115 50  0001 C CNN
 F 3 "~" H 2925 4125 50  0001 C CNN
 	1    2925 4125
@@
 F 0 "R3" H 3593 3421 50  0000 L CNN
 F 1 "100K" H 3593 3330 50  0000 L CNN
-F 2 "Resistor_SMD:R_1206_3216Metric" V 3565 3365 50  0001 C CNN
+F 2 "Resistor_THT:R_Axial_DIN0207_L6.3mm_D2.5mm_P10.16mm_Horizontal" V 3565 3365 50  0001 C CNN
 F 3 "~" H 3525 3375 50  0001 C CNN
 	1    3525 3375
@@
 F 0 "R8" V 7870 3100 50  0000 C CNN
 F 1 "0" V 7961 3100 50  0000 C CNN
-F 2 "Resistor_SMD:R_1206_3216Metric" V 8115 3090 50  0001 C CNN
+F 2 "Resistor_THT:R_Axial_DIN0207_L6.3mm_D2.5mm_P10.16mm_Horizontal" V 8115 3090 50  0001 C CNN
 F 3 "~" H 8075 3100 50  0001 C CNN
 	1    8075 3100
@@
 F 0 "R9" H 8600 3325 50  0000 C CNN
 F 1 "INF" H 8550 3400 50  0000 C CNN
-F 2 "Resistor_SMD:R_1206_3216Metric" V 8415 3340 50  0001 C CNN
+F 2 "Resistor_THT:R_Axial_DIN0207_L6.3mm_D2.5mm_P10.16mm_Horizontal" V 8415 3340 50  0001 C CNN
 F 3 "~" H 8375 3350 50  0001 C CNN
 	1    8375 3350
@@
 F 0 "C6" H 4715 6746 50  0000 L CNN
 F 1 "0.1u" H 4715 6655 50  0000 L CNN
-F 2 "Capacitor_SMD:C_1206_3216Metric" H 4638 6550 50  0001 C CNN
+F 2 "Capacitor_THT:C_Disc_D7.5mm_W4.4mm_P5.00mm" H 4638 6550 50  0001 C CNN
 F 3 "~" H 4600 6700 50  0001 C CNN
 	1    4600 6700

Commit message: Added mounting holes to the Input Signal Conditioner PCB. Also began citation information for ISC documentation.
Parts:
- added H1, H2, H3, H4: MountingHole_Pad, MountingHole:MountingHole_3.2mm_M3_Pad, symbol Mechanical:MountingHole_Pad
Connections:
- net GND: now also H1.1, H2.1, H3.1, H4.1
Changed lines of the file:
@@
 Text Label 3850 3000 0    50   ~ 0
 AMP_IN
+$Comp
+L Mechanical:MountingHole_Pad H1
+U 1 1 5F9CD929
+P 1275 6975
+F 0 "H1" H 1375 6978 50  0000 L CNN
+F 1 "MountingHole_Pad" H 1375 6933 50  0001 L CNN
+F 2 "MountingHole:MountingHole_3.2mm_M3_Pad" H 1275 6975 50  0001 C CNN
+F 3 "~" H 1275 6975 50  0001 C CNN
+	1    1275 6975
+	1    0    0    -1
+$EndComp
+$Comp
+L Mechanical:MountingHole_Pad H2
+U 1 1 5F9CECAE
+P 1650 6975
+F 0 "H2" H 1750 6978 50  0000 L CNN
+F 1 "MountingHole_Pad" H 1750 6933 50  0001 L CNN
+F 2 "MountingHole:MountingHole_3.2mm_M3_Pad" H 1650 6975 50  0001 C CNN
+F 3 "~" H 1650 6975 50  0001 C CNN
+	1    1650 6975
+	1    0    0    -1
+$EndComp
+$Comp
+L Mechanical:MountingHole_Pad H3
+U 1 1 5F9CF11F
+P 2050 6975
+F 0 "H3" H 2150 6978 50  0000 L CNN
+F 1 "MountingHole_Pad" H 2150 6933 50  0001 L CNN
+F 2 "MountingHole:MountingHole_3.2mm_M3_Pad" H 2050 6975 50  0001 C CNN
+F 3 "~" H 2050 6975 50  0001 C CNN
+	1    2050 6975
+	1    0    0    -1
+$EndComp
+$Comp
+L Mechanical:MountingHole_Pad H4
+U 1 1 5F9CF59E
+P 2450 6975
+F 0 "H4" H 2550 6978 50  0000 L CNN
+F 1 "MountingHole_Pad" H 2550 6933 50  0001 L CNN
+F 2 "MountingHole:MountingHole_3.2mm_M3_Pad" H 2450 6975 50  0001 C CNN
+F 3 "~" H 2450 6975 50  0001 C CNN
+	1    2450 6975
+	1    0    0    -1
+$EndComp
+Wire Wire Line
+	1275 7075 1275 7300
+Wire Wire Line
+	1275 7300 1650 7300
+Wire Wire Line
+	2450 7300 2450 7075
+Wire Wire Line
+	2050 7075 2050 7300
+Connection ~ 2050 7300
+Wire Wire Line
+	2050 7300 2450 7300
+Wire Wire Line
+	1650 7075 1650 7300
+Connection ~ 1650 7300
+Wire Wire Line
+	1650 7300 2050 7300
+Wire Wire Line
+	1650 7300 1650 7475
+$Comp
+L power:GND #PWR0102
+U 1 1 5F9D83D0
+P 1650 7475
+F 0 "#PWR0102" H 1650 7225 50  0001 C CNN
+F 1 "GND" H 1655 7302 50  0000 C CNN
+F 2 "" H 1650 7475 50  0001 C CNN
+F 3 "" H 1650 7475 50  0001 C CNN
+	1    1650 7475
+	1    0    0    -1
+$EndComp
 $EndSCHEMATC

Commit message: Made edits suggested by Mark to the ISC pcb. Sent the board for Milling.
Parts:
- added C7: 0.1u, Capacitor_THT:C_Disc_D7.5mm_W4.4mm_P5.00mm, symbol Device:C
Connections:
- net 3.3V: now also C7.2
- net GND: now also C7.1
Changed lines of the file:
@@
 	4825 3475 4825 3400
 Wire Wire Line
-	4825 2800 4825 2600
+	4825 2800 4825 2675
 Text GLabel 4825 2600 1    50   UnSpc ~ 0
 3.3V
@@
 	1    0    0    -1
 $EndComp
+$Comp
+L Device:C C7
+U 1 1 5FA06599
+P 5300 2675
+F 0 "C7" V 5150 2725 50  0000 L CNN
+F 1 "0.1u" V 5225 2725 50  0000 L CNN
+F 2 "Capacitor_THT:C_Disc_D7.5mm_W4.4mm_P5.00mm" H 5338 2525 50  0001 C CNN
+F 3 "~" H 5300 2675 50  0001 C CNN
+	1    5300 2675
+	0    1    1    0
+$EndComp
+Wire Wire Line
+	5150 2675 4825 2675
+Connection ~ 4825 2675
+Wire Wire Line
+	4825 2675 4825 2600
+Wire Wire Line
+	5450 2675 5600 2675
+Wire Wire Line
+	5600 2675 5600 2800
+$Comp
+L power:GND #PWR0103
+U 1 1 5FA0DDC2
+P 5600 2800
+F 0 "#PWR0103" H 5600 2550 50  0001 C CNN
+F 1 "GND" H 5700 2800 50  0000 C CNN
+F 2 "" H 5600 2800 50  0001 C CNN
+F 3 "" H 5600 2800 50  0001 C CNN
+	1    5600 2800
+	1    0    0    -1
+$EndComp

Commit message: Updated an incorrect resistor value on the schematic (resistor R6).
Parts:
- R6: value 11.25K -> 7.68K
Changed lines of the file:
@@
 P 5850 3100
 F 0 "R6" V 5645 3100 50  0000 C CNN
-F 1 "11.25K" V 5736 3100 50  0000 C CNN
+F 1 "7.68K" V 5736 3100 50  0000 C CNN
 F 2 "Resistor_THT:R_Axial_DIN0207_L6.3mm_D2.5mm_P10.16mm_Horizontal" V 5890 3090 50  0001 C CNN
 F 3 "~" H 5850 3100 50  0001 C CNN
