File: Hardware/Boards/Digimuser_Board/Digimuser_Board/Digimuser_Board.sch (KiCad schematic (older format))
At the start: 64 parts, among them J1 Conn_01x01, J10 Conn_01x01, J11 Conn_01x01, J12 Conn_01x01, J2 Conn_01x01, J3 Barrel_Jack_MountingPin, J4 Conn_01x03, J5 Conn_01x03, J6 Conn_01x01, J7 Conn_01x01, J8 Conn_01x01, J9 Conn_01x01, U1 R20407RR02Q, U2 UA78M05IDCYR, U3 MCP6272, U4 Teensy4.0, U5 MCP6271T-E_OT, U6 CS5343-CZZ, U7 CS4344-CZZ

Commit message: Completed most of the PCB layout organization. Still have a lot of work on it.
Parts:
- J1: footprint Connector_PinSocket_2.54mm:PinSocket_1x01_P2.54mm_Vertical -> Connector_PinHeader_2.54mm:PinHeader_1x01_P2.54mm_Vertical
- J10, J11, J12, J6, J7, J8, J9: footprint Connector_Pin:Pin_D1.3mm_L11.0mm_LooseFit -> Connector_PinHeader_2.54mm:PinHeader_1x01_P2.54mm_Vertical
- U4: footprint teensy:Teensy40 -> teensy:Teensy40_HAT
Connections:
- net MLCK is gone; now on net MCLK: U6.4 (MCLK)
- net 3.3V: now also C16.1, C19.1, U4.16 (3V3), U4.31 (3V3), U7.9 (VA); no longer U4.49 (3V3)
- net +9V: now reaches C22.1, J3.1, U2.1 (VIN)
- no-connect marks 35 -> 36
Changed lines of the file:
@@
 $EndComp
-$Comp
-L power:PWR_FLAG #FLG02
-U 1 1 5F936862
-P 9500 5975
-F 0 "#FLG02" H 9500 6050 50  0001 C CNN
-F 1 "PWR_FLAG" H 9500 6148 50  0000 C CNN
-F 2 "" H 9500 5975 50  0001 C CNN
-F 3 "~" H 9500 5975 50  0001 C CNN
-	1    9500 5975
-	1    0    0    -1
-$EndComp
-$Comp
-L power:GND #PWR022
-U 1 1 5F936CB6
-P 9500 6150
-F 0 "#PWR022" H 9500 5900 50  0001 C CNN
-F 1 "GND" H 9505 5977 50  0000 C CNN
-F 2 "" H 9500 6150 50  0001 C CNN
-F 3 "" H 9500 6150 50  0001 C CNN
-	1    9500 6150
-	1    0    0    -1
-$EndComp
-$Comp
-L power:PWR_FLAG #FLG01
-U 1 1 5F93ABBE
-P 9125 6150
-F 0 "#FLG01" H 9125 6225 50  0001 C CNN
-F 1 "PWR_FLAG" H 9125 6323 50  0000 C CNN
-F 2 "" H 9125 6150 50  0001 C CNN
-F 3 "~" H 9125 6150 50  0001 C CNN
-	1    9125 6150
-	-1   0    0    1
-$EndComp
-Text GLabel 9125 5950 1    50   UnSpc ~ 0
-3.3V
-Wire Wire Line
-	9125 6150 9125 5950
-Wire Wire Line
-	9500 6150 9500 5975
 $Comp
 L Connector_Generic:Conn_01x01 J1
@@
 F 0 "J1" H 700 1500 50  0000 L CNN
 F 1 "Conn_01x01" H 400 1150 50  0001 L CNN
-F 2 "Connector_PinSocket_2.54mm:PinSocket_1x01_P2.54mm_Vertical" H 750 1400 50  0001 C CNN
+F 2 "Connector_PinHeader_2.54mm:PinHeader_1x01_P2.54mm_Vertical" H 750 1400 50  0001 C CNN
 F 3 "~" H 750 1400 50  0001 C CNN
 	1    750  1400
@@
 F 0 "U4" H 3775 7790 50  0000 C CNN
 F 1 "Teensy4.0" H 3775 7699 50  0000 C CNN
-F 2 "teensy:Teensy40" H 3375 6375 50  0001 C CNN
+F 2 "teensy:Teensy40_HAT" H 3375 6375 50  0001 C CNN
 F 3 "" H 3375 6375 50  0001 C CNN
 	1    3775 6175
@@
 LRCK
 Text GLabel 8375 1450 0    50   Input ~ 0
-MLCK
-Wire Wire Line
-	8550 1450 8375 1450
+MCLK
 Wire Wire Line
 	8550 1000 7775 1000
@@
 F 0 "J6" V 9950 1900 50  0000 L CNN
 F 1 "Conn_01x01" V 10075 1650 50  0001 L CNN
-F 2 "Connector_Pin:Pin_D1.3mm_L11.0mm_LooseFit" H 9950 2075 50  0001 C CNN
+F 2 "Connector_PinHeader_2.54mm:PinHeader_1x01_P2.54mm_Vertical" H 9950 2075 50  0001 C CNN
 F 3 "~" H 9950 2075 50  0001 C CNN
 	1    9950 2075
@@
 F 0 "J7" H 10525 3275 50  0000 L CNN
 F 1 "Conn_01x01" V 10675 2975 50  0001 L CNN
-F 2 "Connector_Pin:Pin_D1.3mm_L11.0mm_LooseFit" H 10550 3400 50  0001 C CNN
+F 2 "Connector_PinHeader_2.54mm:PinHeader_1x01_P2.54mm_Vertical" H 10550 3400 50  0001 C CNN
 F 3 "~" H 10550 3400 50  0001 C CNN
 	1    10550 3400
@@
 Text Notes 8000 5275 0    50   ~ 0
 SOT-23-5 Package
-Wire Wire Line
-	4875 7225 5100 7225
 Wire Wire Line
 	5175 5525 4875 5525
@@
 L power:GND #PWR012
 U 1 1 5FD514D9
-P 5100 7225
-F 0 "#PWR012" H 5100 6975 50  0001 C CNN
-F 1 "GND" H 5200 7100 50  0000 C CNN
-F 2 "" H 5100 7225 50  0001 C CNN
-F 3 "" H 5100 7225 50  0001 C CNN
-	1    5100 7225
+P 5200 7225
+F 0 "#PWR012" H 5200 6975 50  0001 C CNN
+F 1 "GND" H 5300 7100 50  0000 C CNN
+F 2 "" H 5200 7225 50  0001 C CNN
+F 3 "" H 5200 7225 50  0001 C CNN
+	1    5200 7225
 	1    0    0    -1
 $EndComp
@@
 $EndComp
 Wire Wire Line
-	4875 5325 5175 5325
-Text GLabel 5175 5325 2    50   UnSpc ~ 0
-3.3V
-Wire Wire Line
 	2425 4825 2425 4875
 Wire Wire Line
@@
 	1    0    0    -1
 $EndComp
-NoConn ~ 4875 7325
 $Comp
 L ‎R20407RR02Q‎_ROT_SWITCH:R20407RR02Q U1
@@
 F 0 "J11" H 9900 5200 50  0000 L CNN
 F 1 "Conn_01x01" V 10050 4900 50  0001 L CNN
-F 2 "Connector_Pin:Pin_D1.3mm_L11.0mm_LooseFit" H 9925 5325 50  0001 C CNN
+F 2 "Connector_PinHeader_2.54mm:PinHeader_1x01_P2.54mm_Vertical" H 9925 5325 50  0001 C CNN
 F 3 "~" H 9925 5325 50  0001 C CNN
 	1    9925 5325
@@
 F 0 "J12" H 10475 4925 50  0000 L CNN
 F 1 "Conn_01x01" V 10625 4625 50  0001 L CNN
-F 2 "Connector_Pin:Pin_D1.3mm_L11.0mm_LooseFit" H 10500 5050 50  0001 C CNN
+F 2 "Connector_PinHeader_2.54mm:PinHeader_1x01_P2.54mm_Vertical" H 10500 5050 50  0001 C CNN
 F 3 "~" H 10500 5050 50  0001 C CNN
 	1    10500 5050
@@
 F 0 "J9" V 6125 7025 50  0000 L CNN
 F 1 "Conn_01x01" V 6400 6700 50  0001 L CNN
-F 2 "Connector_Pin:Pin_D1.3mm_L11.0mm_LooseFit" H 6275 7125 50  0001 C CNN
+F 2 "Connector_PinHeader_2.54mm:PinHeader_1x01_P2.54mm_Vertical" H 6275 7125 50  0001 C CNN
 F 3 "~" H 6275 7125 50  0001 C CNN
 	1    6275 7125
@@
 F 0 "J10" V 6400 7025 50  0000 L CNN
 F 1 "Conn_01x01" V 6675 6700 50  0001 L CNN
-F 2 "Connector_Pin:Pin_D1.3mm_L11.0mm_LooseFit" H 6550 7125 50  0001 C CNN
+F 2 "Connector_PinHeader_2.54mm:PinHeader_1x01_P2.54mm_Vertical" H 6550 7125 50  0001 C CNN
 F 3 "~" H 6550 7125 50  0001 C CNN
 	1    6550 7125
@@
 F 0 "J8" V 6000 6975 50  0000 L CNN
 F 1 "Conn_01x01" V 6125 6700 50  0001 L CNN
-F 2 "Connector_Pin:Pin_D1.3mm_L11.0mm_LooseFit" H 6000 7125 50  0001 C CNN
+F 2 "Connector_PinHeader_2.54mm:PinHeader_1x01_P2.54mm_Vertical" H 6000 7125 50  0001 C CNN
 F 3 "~" H 6000 7125 50  0001 C CNN
 	1    6000 7125
@@
 	1    0    0    -1
 $EndComp
+Text Label 1775 3850 0    50   ~ 0
++9V
+Text GLabel 4925 7325 2    50   UnSpc ~ 0
+3.3V
+Wire Wire Line
+	4875 7225 5200 7225
+Wire Wire Line
+	4875 7325 4925 7325
+Text GLabel 2525 6325 0    50   UnSpc ~ 0
+3.3V
+Wire Wire Line
+	2675 6325 2525 6325
+Wire Wire Line
+	8550 1450 8375 1450
+NoConn ~ 2675 5125
+Text Label 9025 5875 0    50   ~ 0
++9V
+$Comp
+L power:PWR_FLAG #FLG0101
+U 1 1 5FD138D1
+P 9025 6100
+F 0 "#FLG0101" H 9025 6175 50  0001 C CNN
+F 1 "PWR_FLAG" H 9025 6273 50  0000 C CNN
+F 2 "" H 9025 6100 50  0001 C CNN
+F 3 "~" H 9025 6100 50  0001 C CNN
+	1    9025 6100
+	-1   0    0    1
+$EndComp
+Wire Wire Line
+	9025 6100 9025 5875
+Text GLabel 10675 2850 1    50   Input ~ 0
+3.3V
+Wire Wire Line
+	10675 2950 10675 2850
+Connection ~ 10675 2950
+NoConn ~ 4875 5325
 $EndSCHEMATC

Commit message: Continued PCB layout.
Parts:
- C13: footprint Capacitor_THT:CP_Radial_D6.3mm_P2.50mm -> Capacitor_THT:C_Axial_L5.1mm_D3.1mm_P7.50mm_Horizontal
- U1: footprint Connector_PinSocket_2.54mm:PinSocket_1x04_P2.54mm_Vertical -> Connector_PinSocket_2.54mm:PinSocket_1x05_P2.54mm_Vertical
Changed lines of the file:
@@
 Connection ~ 8425 3550
-$Comp
-L Device:CP1 C13
-U 1 1 5FB97996
-P 9925 3700
-F 0 "C13" H 10040 3746 50  0000 L CNN
-F 1 "10u" H 10040 3655 50  0000 L CNN
-F 2 "Capacitor_THT:CP_Radial_D6.3mm_P2.50mm" H 9925 3700 50  0001 C CNN
-F 3 "~" H 9925 3700 50  0001 C CNN
-	1    9925 3700
-	1    0    0    -1
-$EndComp
 $Comp
 L Device:C C16
@@
 F 0 "U1" H 933 6950 50  0000 C CNN
 F 1 "R20407RR02Q" H 933 6859 50  0000 C CNN
-F 2 "Connector_PinSocket_2.54mm:PinSocket_1x04_P2.54mm_Vertical" H 900 6725 50  0001 C CNN
+F 2 "Connector_PinSocket_2.54mm:PinSocket_1x05_P2.54mm_Vertical" H 900 6725 50  0001 C CNN
 F 3 "" H 900 6725 50  0001 C CNN
 	1    900  6725
@@
 Connection ~ 10675 2950
 NoConn ~ 4875 5325
+$Comp
+L Device:CP1 C13
+U 1 1 5FB97996
+P 9925 3700
+F 0 "C13" H 10040 3746 50  0000 L CNN
+F 1 "10u" H 10040 3655 50  0000 L CNN
+F 2 "Capacitor_THT:C_Axial_L5.1mm_D3.1mm_P7.50mm_Horizontal" H 9925 3700 50  0001 C CNN
+F 3 "~" H 9925 3700 50  0001 C CNN
+	1    9925 3700
+	1    0    0    -1
+$EndComp
 $EndSCHEMATC

Commit message: Finished the first revision of the PCB layout. Needs reviewing.
Parts:
- J1, J10, J11, J12, J6, J7, J8, J9: footprint Connector_PinHeader_2.54mm:PinHeader_1x01_P2.54mm_Vertical -> Custom_Connectors:PinHeader_2.54mm_1x01_P2.54mm
- J2: footprint Connector_PinSocket_2.54mm:PinSocket_1x01_P2.54mm_Vertical -> Custom_Connectors:PinHeader_2.54mm_1x01_P2.54mm
- J4, J5: footprint Connector_PinHeader_2.54mm:PinHeader_1x03_P2.54mm_Vertical -> Custom_Connectors:PinHeader_2.54mm_1x03_P2.54mm
- U1: footprint Connector_PinSocket_2.54mm:PinSocket_1x05_P2.54mm_Vertical -> Custom_Connectors:R20407RR02Q
Changed lines of the file:
@@
 F 0 "J4" H 2030 1442 50  0000 L CNN
 F 1 "Conn_01x03" H 2030 1351 50  0001 L CNN
-F 2 "Connector_PinHeader_2.54mm:PinHeader_1x03_P2.54mm_Vertical" H 1950 1400 50  0001 C CNN
+F 2 "Custom_Connectors:PinHeader_2.54mm_1x03_P2.54mm" H 1950 1400 50  0001 C CNN
 F 3 "~" H 1950 1400 50  0001 C CNN
 	1    1950 1400
@@
 F 0 "J1" H 700 1500 50  0000 L CNN
 F 1 "Conn_01x01" H 400 1150 50  0001 L CNN
-F 2 "Connector_PinHeader_2.54mm:PinHeader_1x01_P2.54mm_Vertical" H 750 1400 50  0001 C CNN
+F 2 "Custom_Connectors:PinHeader_2.54mm_1x01_P2.54mm" H 750 1400 50  0001 C CNN
 F 3 "~" H 750 1400 50  0001 C CNN
 	1    750  1400
@@
 F 0 "J2" V 750 1675 50  0000 L CNN
 F 1 "Conn_01x01" V 875 1425 50  0001 L CNN
-F 2 "Connector_PinSocket_2.54mm:PinSocket_1x01_P2.54mm_Vertical" H 750 1850 50  0001 C CNN
+F 2 "Custom_Connectors:PinHeader_2.54mm_1x01_P2.54mm" H 750 1850 50  0001 C CNN
 F 3 "~" H 750 1850 50  0001 C CNN
 	1    750  1850
@@
 F 0 "J6" V 9950 1900 50  0000 L CNN
 F 1 "Conn_01x01" V 10075 1650 50  0001 L CNN
-F 2 "Connector_PinHeader_2.54mm:PinHeader_1x01_P2.54mm_Vertical" H 9950 2075 50  0001 C CNN
+F 2 "Custom_Connectors:PinHeader_2.54mm_1x01_P2.54mm" H 9950 2075 50  0001 C CNN
 F 3 "~" H 9950 2075 50  0001 C CNN
 	1    9950 2075
@@
 F 0 "J7" H 10525 3275 50  0000 L CNN
 F 1 "Conn_01x01" V 10675 2975 50  0001 L CNN
-F 2 "Connector_PinHeader_2.54mm:PinHeader_1x01_P2.54mm_Vertical" H 10550 3400 50  0001 C CNN
+F 2 "Custom_Connectors:PinHeader_2.54mm_1x01_P2.54mm" H 10550 3400 50  0001 C CNN
 F 3 "~" H 10550 3400 50  0001 C CNN
 	1    10550 3400
@@
 F 0 "J5" H 9630 4992 50  0000 L CNN
 F 1 "Conn_01x03" H 9630 4901 50  0001 L CNN
-F 2 "Connector_PinHeader_2.54mm:PinHeader_1x03_P2.54mm_Vertical" H 9550 4950 50  0001 C CNN
+F 2 "Custom_Connectors:PinHeader_2.54mm_1x03_P2.54mm" H 9550 4950 50  0001 C CNN
 F 3 "~" H 9550 4950 50  0001 C CNN
 	1    9550 4950
@@
 F 0 "U1" H 933 6950 50  0000 C CNN
 F 1 "R20407RR02Q" H 933 6859 50  0000 C CNN
-F 2 "Connector_PinSocket_2.54mm:PinSocket_1x05_P2.54mm_Vertical" H 900 6725 50  0001 C CNN
+F 2 "Custom_Connectors:R20407RR02Q" H 900 6725 50  0001 C CNN
 F 3 "" H 900 6725 50  0001 C CNN
 	1    900  6725
@@
 F 0 "J11" H 9900 5200 50  0000 L CNN
 F 1 "Conn_01x01" V 10050 4900 50  0001 L CNN
-F 2 "Connector_PinHeader_2.54mm:PinHeader_1x01_P2.54mm_Vertical" H 9925 5325 50  0001 C CNN
+F 2 "Custom_Connectors:PinHeader_2.54mm_1x01_P2.54mm" H 9925 5325 50  0001 C CNN
 F 3 "~" H 9925 5325 50  0001 C CNN
 	1    9925 5325
@@
 F 0 "J12" H 10475 4925 50  0000 L CNN
 F 1 "Conn_01x01" V 10625 4625 50  0001 L CNN
-F 2 "Connector_PinHeader_2.54mm:PinHeader_1x01_P2.54mm_Vertical" H 10500 5050 50  0001 C CNN
+F 2 "Custom_Connectors:PinHeader_2.54mm_1x01_P2.54mm" H 10500 5050 50  0001 C CNN
 F 3 "~" H 10500 5050 50  0001 C CNN
 	1    10500 5050
@@
 F 0 "J9" V 6125 7025 50  0000 L CNN
 F 1 "Conn_01x01" V 6400 6700 50  0001 L CNN
-F 2 "Connector_PinHeader_2.54mm:PinHeader_1x01_P2.54mm_Vertical" H 6275 7125 50  0001 C CNN
+F 2 "Custom_Connectors:PinHeader_2.54mm_1x01_P2.54mm" H 6275 7125 50  0001 C CNN
 F 3 "~" H 6275 7125 50  0001 C CNN
 	1    6275 7125
@@
 F 0 "J10" V 6400 7025 50  0000 L CNN
 F 1 "Conn_01x01" V 6675 6700 50  0001 L CNN
-F 2 "Connector_PinHeader_2.54mm:PinHeader_1x01_P2.54mm_Vertical" H 6550 7125 50  0001 C CNN
+F 2 "Custom_Connectors:PinHeader_2.54mm_1x01_P2.54mm" H 6550 7125 50  0001 C CNN
 F 3 "~" H 6550 7125 50  0001 C CNN
 	1    6550 7125
@@
 F 0 "J8" V 6000 6975 50  0000 L CNN
 F 1 "Conn_01x01" V 6125 6700 50  0001 L CNN
-F 2 "Connector_PinHeader_2.54mm:PinHeader_1x01_P2.54mm_Vertical" H 6000 7125 50  0001 C CNN
+F 2 "Custom_Connectors:PinHeader_2.54mm_1x01_P2.54mm" H 6000 7125 50  0001 C CNN
 F 3 "~" H 6000 7125 50  0001 C CNN
 	1    6000 7125
