File: Hardware/Boards/Digimuser_Board/Digimuser_Board/Digimuser_Board.kicad_pcb (KiCad board)
At the start: 2 copper layers, 60.2 x 38.7 mm, 74 parts, among them J1 Conn_01x01, J10 Conn_01x01, J11 Conn_01x01, J12 Conn_01x01, J13 Conn_01x01, J14 Conn_01x01, J15 Conn_01x01, J2 Conn_01x01, J3 Barrel_Jack_MountingPin, J4 Conn_01x03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

Commit message: Finished final details for first prototype.
Parts:
- C24, C25: value 3.9n -> 3.3n
- U6: value CIR-TSSOP-10 -> CS5343-CZZ
- U7: value CIR-TSSOP-10 -> CS4344-CZZ
